File: tuto_usb-c/STM32.kicad_sch (KiCad schematic)
At the start: 25 parts, among them J2 Conn_01x06, J301 Conn_ST_STDC14, J4 Conn_01x06, U3 STM32G431KBT6, Y301 Crystal_GND24_Small

Commit message: modif routing - add gng plane
Parts:
- Y301: footprint (none) -> Crystal:Crystal_SMD_0603-4Pin_6.0x3.5mm
Changed lines of the file:
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@@
 			)
 		)
-		(property "Footprint" ""
+		(property "Footprint" "Crystal:Crystal_SMD_0603-4Pin_6.0x3.5mm"
 			(at 102.87 74.93 0)
 			(effects
