File: tuto_usb-c/USB.kicad_sch (KiCad schematic)
At the start: 9 parts, among them J202 USB_C_Receptacle_USB2.0_16P, U201 USBLC6-2SC6, U202 MCP1802x-xx02xOT

Commit message: modif routing - add gng plane
Parts:
- C1: footprint Connector_USB:USB_C_Receptacle_HRO_TYPE-C-31-M-12 -> Capacitor_SMD:C_0603_1608Metric_Pad1.08x0.95mm_HandSolder
- F201: footprint (none) -> Fuse:Fuse_1206_3216Metric
- FB202: footprint (none) -> Inductor_SMD:L_0805_2012Metric
- J202: footprint (none) -> Connector_USB:USB_C_Receptacle_HRO_TYPE-C-31-M-12
Changed lines of the file:
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@@
 			)
 		)
-		(property "Footprint" ""
+		(property "Footprint" "Inductor_SMD:L_0805_2012Metric"
 			(at 215.9 140.208 90)
 			(effects
@@
 			)
 		)
-		(property "Footprint" ""
+		(property "Footprint" "Fuse:Fuse_1206_3216Metric"
 			(at 233.68 137.16 0)
 			(effects
@@
 			)
 		)
-		(property "Footprint" "Connector_USB:USB_C_Receptacle_HRO_TYPE-C-31-M-12"
+		(property "Footprint" "Capacitor_SMD:C_0603_1608Metric_Pad1.08x0.95mm_HandSolder"
 			(at 207.01 64.77 0)
 			(effects
@@
 			)
 		)
-		(property "Footprint" ""
+		(property "Footprint" "Connector_USB:USB_C_Receptacle_HRO_TYPE-C-31-M-12"
 			(at 50.8 48.26 0)
 			(effects
